Commit message: Update model.urdf

File: objects/ycb_objects/YcbScissors/model.urdf (robot description, URDF)
Before this commit: robot model.urdf, 1 links, 0 joints
Links:
- link baseLink: mass .182 -> .300; geometry collision mesh filename=collision_vhacd.obj scale=1 1.5 2; visual mesh filename=textured_simple_reoriented.obj scale=1 1.5 2
